File: Amplifier/Amplifier.kicad_pcb (KiCad board)
At the start: 2 copper layers, 55 x 52 mm, 62 parts, among them J7 Conn_01x14_MountingPin, Q3 2N7002, U13 AD40xxBRMZ, U14 LP5907MFX-1.8, U16 LTC6268xS8, U17 ADG1219BRMZ, U2 LMP7721, U5 OPA2192IDR, U6 ADA4940-1xCP

Commit message: Transition Amplifier to discrete pogo pins on F.Cu
Update Amplifier schematic and PCB to use 12 discrete single-pin
SMT pogo pins (P1..P12) placed on F.Cu (top layer) alongside active
components for a single-sided board assembly. Update J_PAD1 to use
PogoPin_Target_Landing_1Pin_Guarded and align test assertions.

Co-authored-by: google-labs-jules[bot] <161369871+google-labs-jules[bot]@users.noreply.github.com>
Parts:
- removed J_POGO1: PogoPin_SpringHeader_6Pin_Cis, footprints:PogoPin_SpringHeader_6Pin_Cis
- removed J_POGO2: PogoPin_SpringHeader_6Pin_Trans, footprints:PogoPin_SpringHeader_6Pin_Trans
- added P1: PogoPin_MillMax_SMT_1Pin, footprints:PogoPin_MillMax_SMT_1Pin, F.Cu at (146.5, 42.5)
- added P10: PogoPin_MillMax_SMT_1Pin, footprints:PogoPin_MillMax_SMT_1Pin, F.Cu at (167.5, 73.5)
- added P11: PogoPin_MillMax_SMT_1Pin, footprints:PogoPin_MillMax_SMT_1Pin, F.Cu at (176.5, 73.5)
- added P12: PogoPin_MillMax_SMT_1Pin, footprints:PogoPin_MillMax_SMT_1Pin, F.Cu at (182.5, 74.5)
- added P2: PogoPin_MillMax_SMT_1Pin_Guarded, footprints:PogoPin_MillMax_SMT_1Pin_Guarded, F.Cu at (154.5, 43.5)
- added P3: PogoPin_MillMax_SMT_1Pin, footprints:PogoPin_MillMax_SMT_1Pin, F.Cu at (158.5, 43.5)
- added P4: PogoPin_MillMax_SMT_1Pin, footprints:PogoPin_MillMax_SMT_1Pin, F.Cu at (168.5, 43.5)
- added P5: PogoPin_MillMax_SMT_1Pin_Guarded, footprints:PogoPin_MillMax_SMT_1Pin_Guarded, F.Cu at (172.5, 43.5)
- added P6: PogoPin_MillMax_SMT_1Pin, footprints:PogoPin_MillMax_SMT_1Pin, F.Cu at (176.5, 43.5)
- added P7: PogoPin_MillMax_SMT_1Pin, footprints:PogoPin_MillMax_SMT_1Pin, F.Cu at (146.5, 74.5)
- added P8: PogoPin_MillMax_SMT_1Pin, footprints:PogoPin_MillMax_SMT_1Pin, F.Cu at (154.5, 73.5)
- added P9: PogoPin_MillMax_SMT_1Pin, footprints:PogoPin_MillMax_SMT_1Pin, F.Cu at (160.5, 73.5)
- J_PAD1: value Concentric_Interposer_Mating_Pad -> PogoPin_Target_Landing_1Pin_Guarded; footprint footprints:Concentric_Interposer_Mating_Pad -> footprints:PogoPin_Target_Landing_1Pin_Guarded; moved to F.Cu
