File: Amplifier/Amplifier.kicad_sch (KiCad schematic)
At the start: 68 parts, among them J7 Conn_01x14_MountingPin, Q3 2N7002, U13 AD40xxBRMZ, U14 LP5907MFX-1.8, U16 LTC6268xS8, U17 ADG1219BRMZ, U2 LMP7721, U5 OPA2192IDR, U6 ADA4940-1xCP

Commit message: Transition Amplifier to discrete pogo pins on F.Cu
Update Amplifier schematic and PCB to use 12 discrete single-pin
SMT pogo pins (P1..P12) placed on F.Cu (top layer) alongside active
components for a single-sided board assembly. Update J_PAD1 to use
PogoPin_Target_Landing_1Pin_Guarded and align test assertions.

Co-authored-by: google-labs-jules[bot] <161369871+google-labs-jules[bot]@users.noreply.github.com>
Parts:
- removed J_POGO1: PogoPin_SpringHeader_6Pin_Cis, footprints:PogoPin_SpringHeader_6Pin_Cis, symbol MR1:PogoPin_SpringHeader_6Pin_Cis
- removed J_POGO2: PogoPin_SpringHeader_6Pin_Trans, footprints:PogoPin_SpringHeader_6Pin_Trans, symbol MR1:PogoPin_SpringHeader_6Pin_Trans
- added J_PAD1: PogoPin_Target_Landing_1Pin_Guarded, footprints:PogoPin_Target_Landing_1Pin_Guarded, symbol MR1:PogoPin_Target_Landing_1Pin_Guarded
- added P1, P10, P11, P12, P3, P4, P6, P7, P8, P9: PogoPin_MillMax_SMT_1Pin, footprints:PogoPin_MillMax_SMT_1Pin, symbol MR1:PogoPin_MillMax_SMT_1Pin
- added P2, P5: PogoPin_MillMax_SMT_1Pin_Guarded, footprints:PogoPin_MillMax_SMT_1Pin_Guarded, symbol MR1:PogoPin_MillMax_SMT_1Pin_Guarded
Connections:
- net >PORE_AMP: now also J_PAD1.2 (GUARD), P9.1 (PIN)
- net CE_GNDA: now also P7.1 (PIN)
- net GNDA: now also P10.1 (PIN)
- net GUARD: now also J_PAD1.1 (SIG), P4.1 (PIN), P5.1 (SIG), P6.1 (PIN)
- net GUARD_WIDE: now also P2.1 (SIG), P3.1 (PIN)
- net RE_TRANS: now also P8.1 (PIN)
- net R_WEEP_LIM: now also P11.1 (PIN)
- net WS_CIS: now also P5.2 (GUARD)
- net WS_CIS_WIDE: now also P2.2 (GUARD)
- new net GNDA_SHLD: P1.1 (PIN)
- new net GNDA_WEEP: P12.1 (PIN)
